Commit message: ~

File: rostest/src/urdf_tutorial/urdf/03-origins.urdf (robot description, URDF)
Before this commit: robot origins, 2 links, 1 joints
Joints:
- joint base_to_right_leg: origin xyz=0 0 0 -> xyz=0 -0.22 0.25

File: rostest/src/urdf_tutorial/urdf/08-macroed.urdf.xacro (robot description, xacro)
@@ -7,5 +7,5 @@
   <xacro:property name="baselen" value="0.4" />
   <xacro:property name="wheeldiam" value="0.07" />
-  <xacro:property name="pi" value="3.1415" />
+  <!-- <xacro:property name="pi" value="3.1415" /> -->
   <material name="blue">
     <color rgba="0 0 0.8 1"/>
@@ -35,5 +35,5 @@
       </geometry>
     </collision>
-    <xacro:default_inertial mass="10"/>
+    <!-- <xacro:default_inertial mass="10"/> -->
   </link>
   <xacro:macro name="wheel" params="prefix suffix reflect">
